File: _autosave-veffy.kicad_sch (KiCad schematic)
At the start: 37 parts, among them J1 SWD, SW1 SW_Push, U1 ATSAMD21G18A-A, U2 ADF4112BCPZ, U3 SA612AN/01_112, U4 MC3361, U5 LM386, U6 LM358_DFN

Commit message: worked on the output AMP stuff
Connections:
- net PRE_AMP: now also U6.1; no longer U5.5
Other:
- moved on the sheet: U6A
Changed lines of the file:
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@@
+		)
+	)
+	(global_label "PRE_AMP"
+		(shape input)
+		(at 189.23 138.43 0)
+		(fields_autoplaced yes)
+		(effects
+			(font
+				(size 1.27 1.27)
+			)
+			(justify left)
+		)
+		(property "Intersheetrefs" "${INTERSHEET_REFS}"
+			(at 200.6818 138.43 0)
+			(hide yes)
+			(show_name no)
+			(do_not_autoplace no)
+			(effects
+				(font
+					(size 1.27 1.27)
+				)
+				(justify left)
+			)
 		)
 	)
@@
 		(property "Intersheetrefs" "${INTERSHEET_REFS}"
 			(at 167.64 95.6347 90)
-			(hide yes)
-			(show_name no)
-			(do_not_autoplace no)
-			(effects
-				(font
-					(size 1.27 1.27)
-				)
-				(justify right)
-			)
-		)
-	)
-	(global_label "PRE_AMP"
-		(shape input)
-		(at 160.02 123.19 270)
-		(fields_autoplaced yes)
-		(effects
-			(font
-				(size 1.27 1.27)
-			)
-			(justify right)
-		)
-		(property "Intersheetrefs" "${INTERSHEET_REFS}"
-			(at 160.02 134.6418 90)
 			(hide yes)
 			(show_name no)
@@
 	(symbol
 		(lib_id "Amplifier_Operational:LM358_DFN")
-		(at 177.8 138.43 0)
+		(at 181.61 138.43 0)
 		(unit 1)
 		(body_style 1)
@@
 		(fields_autoplaced yes)
 		(property "Reference" "U6"
-			(at 177.8 128.27 0)
+			(at 181.61 128.27 0)
 			(show_name no)
 			(do_not_autoplace no)
@@
 		)
 		(property "Value" "LM358_DFN"
-			(at 177.8 130.81 0)
+			(at 181.61 130.81 0)
 			(show_name no)
 			(do_not_autoplace no)
@@
 		)
 		(property "Footprint" "Package_CSP:LFCSP-8_2x2mm_P0.5mm"
-			(at 177.8 138.43 0)
+			(at 181.61 138.43 0)
 			(hide yes)
 			(show_name no)
@@
 		)
 		(property "Datasheet" "www.st.com/resource/en/datasheet/lm358.pdf"
-			(at 177.8 138.43 0)
+			(at 181.61 138.43 0)
 			(hide yes)
 			(show_name no)
@@
 		)
 		(property "Description" "Low-Power, Dual Operational Amplifiers, DFN-8"
-			(at 177.8 138.43 0)
-			(hide yes)
-			(show_name no)
+			(at 181.61 138.43 0)
+			(hide yes)
+			(show_name no)
