File: veffy.kicad_pcb (KiCad board)
At the start: 4 copper layers, 142 parts, among them CN1 XH-2AW_C2908611, J1 SWD, J2 Conn_Coaxial, J3 USB_C_Receptacle_USB2.0_14P, Q1 2N7002, Q2 BFR93A, Q3 2N7002, Q4 BFR93AE6327HTSA1, SW1 SW_Push, SW2 SW_Push, U1 ATSAMD21G18A-A, U10 MC34063AD, U11 AP2112K-3.3, U4 MC3361, U6 LM358_DFN, U7 AD9834, U8 QPA9510, U9 MCP73831-2-OT, Y2 C7527392

Commit message: mic amp fixes
Parts:
- removed L6: 1uH, Inductor_SMD:L_0603_1608Metric
- added C64: 1nF, Capacitor_SMD:C_0603_1608Metric, F.Cu at (135.5, 127.8)
- added C65: 2-10pF, Capacitor_SMD:C_Trimmer_Murata_TZB4-A, F.Cu at (129.2, 126.8)
- added C66: 2-10pF, Capacitor_SMD:C_Trimmer_Murata_TZB4-A, F.Cu at (129.2, 132.3)
- added C67: 2-10pF, Capacitor_SMD:C_Trimmer_Murata_TZB4-A, F.Cu at (129.2, 137.9)
- added D1: SMV1236-079LF, LCSC:SC-79_L1.2-W0.8-LS1.6-RD, F.Cu at (135.1, 130.1)
- added R36: 680, Resistor_SMD:R_0603_1608Metric_Pad0.98x0.95mm_HandSolder, F.Cu at (135.6, 125.3)
- C7: value 100pF -> 10pF
- CN1: footprint LCSC:CONN-TH_XH-2AW_C2908611 -> Connector_PinHeader_2.00mm:PinHeader_1x02_P2.00mm_Vertical_SMD_Pin1Right
- J1: footprint Connector_PinHeader_2.54mm:PinHeader_1x04_P2.54mm_Vertical_SMD_Pin1Left -> Connector_PinHeader_1.00mm:PinHeader_1x05_P1.00mm_Vertical
- SW1, SW2: footprint Button_Switch_SMD:SW_Push_1P1T_NO_CK_PTS125Sx43SMTR -> Button_Switch_SMD:SW_MEC_5GSH9
- moved R27 108.1 mm to (199.3, 137.6), turned to 90 degrees
- moved R28 105.6 mm to (197.8, 137.6), turned to -90 degrees
- moved J3 104.5 mm to (198.4, 143.8)
- moved CN1 97.2 mm to (181.2, 143.3)
- moved U9 86.2 mm to (186.2, 144.1)
- moved FB1 48.6 mm to (204.4, 143.2), turned to 90 degrees
- moved C51 42.8 mm to (189.9, 145.1), turned to 180 degrees
- moved C52 38.2 mm to (185.7, 141.7)
- moved R29 32.4 mm to (188.2, 140.9), turned to -90 degrees
Connections:
- C7 pad 2: Net-(U3-INPUTB) -> INPUTB
- R14 pad 1: Net-(U7-IOUT) -> Net-(R14-Pad1)
Routing:
- net Net-(J3-SHIELD): track 0.00 -> 21.4 mm
- net VBUS: track 0.00 -> 19.7 mm
- net BAT+: track 0.00 -> 10.8 mm
- net AGND: track 0.00 -> 5.21 mm, vias 0 -> 7
- net Net-(J3-CC2): track 0.00 -> 2.28 mm
- net Net-(J3-CC1): track 0.00 -> 2.10 mm
- net Net-(U9-PROG): track 0.00 -> 1.69 mm
- added copper zone on B.Cu, net AGND
- added copper zone on F.Cu, net AGND
- added copper zone on In1.Cu, net DVDD

Commit message: fixing the T/R switch and updating some footprints
Parts:
- added C68: 1uF, Capacitor_SMD:C_0603_1608Metric_Pad1.08x0.95mm_HandSolder, F.Cu at (149.6, 109.6)
- added C69: 10nF, Capacitor_SMD:C_0603_1608Metric_Pad1.08x0.95mm_HandSolder, F.Cu at (149.6, 112.1)
- added R37: 1K, Resistor_SMD:R_0603_1608Metric_Pad0.98x0.95mm_HandSolder, F.Cu at (149.6, 114.6)
- C21: value 10uF -> 4.7uF
- C25: value 1uF -> 1nF
- J1: footprint Connector_PinHeader_1.00mm:PinHeader_1x05_P1.00mm_Vertical -> Connector_PinHeader_1.00mm:PinHeader_1x05_P1.00mm_Vertical_SMD_Pin1Right
- R6: value 15K -> 47K
- U6: value LM358_DFN -> TLV9062IDSGR
Connections:
- C21 pad 1: Net-(MK1-+) -> Net-(C21-Pad1)
- C21 pad 2: PRE_AMP -> AGND
- C25 pad 1: MIC_PREAMP -> Net-(U6B--)
- C25 pad 2: Net-(U6B-+) -> PRE_AMP
- R7 pad 2: AGND -> Net-(C21-Pad1)
- U1 pad 9: unconnected-(U1-PA04-Pad9) -> Net-(U1-PA04)
- U6 pad 5: Net-(U6B-+) -> MIC_PREAMP
